Commit message: change tool orientation for demo robot

File: taskspace_control_examples/urdf/robot6R_macro.xacro (robot description, xacro)
@@ -216,4 +216,10 @@
       </visual>
     </link>
+    <link name="${prefix}tool"/>
+    <joint name="${prefix}tool_joint" type="fixed">
+      <origin xyz="0 0 0" rpy="${-pi/2} ${-pi/2} 0"/>
+      <parent link="${prefix}tool0"/>
+      <child link="${prefix}tool"/>
+    </joint>
   </xacro:macro>
 </robot>

Commit message: add 7R robot to examples

File: taskspace_control_examples/urdf/robot6R_macro.xacro (robot description, xacro)
@@ -100,5 +100,5 @@
         <origin xyz="0 0 0" rpy="${pi / 2.0} 0 0" />
         <geometry>
-                <cylinder length="${joint_length}" radius="${joint_radius}"/>
+          <cylinder length="${joint_length}" radius="${joint_radius}"/>
         </geometry>
         <material name="grey"/>
@@ -107,5 +107,5 @@
         <origin xyz="0 ${link4_length / 2.0} 0" rpy="${pi / 2.0} 0 0" />
         <geometry>
-                <cylinder length="${link4_length}" radius="${link_radius}"/>
+          <cylinder length="${link4_length}" radius="${link_radius}"/>
         </geometry>
         <material name="grey"/>
@@ -114,5 +114,5 @@
         <origin xyz="0 ${link4_length} 0" rpy="0 0 0" />
         <geometry>
-                <cylinder length="${joint_length}" radius="${joint_radius}"/>
+          <cylinder length="${joint_length}" radius="${joint_radius}"/>
         </geometry>
         <material name="grey"/>

File: taskspace_control_examples/urdf/robot7R.xacro (robot description, xacro)
@@ -1,10 +1,10 @@
 <?xml version="1.0"?>
-<robot name="robot6R" xmlns:xacro="http://ros.org/wiki/xacro">
+<robot name="robot7R" xmlns:xacro="http://ros.org/wiki/xacro">
   <xacro:arg name="prefix" default=""/>
-  <xacro:include filename="$(find taskspace_control_examples)/urdf/robot6R_macro.xacro"/>
-  <xacro:robot6R_macro prefix="$(arg prefix)"/>
+  <xacro:include filename="$(find taskspace_control_examples)/urdf/robot7R_macro.xacro"/>
+  <xacro:robot7R_macro prefix="$(arg prefix)"/>
   <!-- colors -->
-  <material name="grey">
-    <color rgba="0.7 0.7 0.7 1.0"/>
+  <material name="cream">
+    <color rgba="1.0 0.99 0.81 1.0"/>
   </material>
   <!-- Connect to world -->
