Commit message: add missing prefix tag in link7 urdf

File: taskspace_control_examples/urdf/robot7R_macro.xacro (robot description, xacro)
@@ -122,5 +122,5 @@
       </visual>
     </link>
-    <link name="link7">
+    <link name="${prefix}link7">
       <visual name="joint7">
         <origin xyz="0 0 0" rpy="0 0 0" />
